File: eagle/CR78-SD.brd (EAGLE design)
At the start: 100 x 80 mm, 39 parts, among them Q1 2N3904, Q2 2N3904, Q4 2N3904, Q6 2N3904, Q7 2N3904

Commit message: more schemo
Parts:
- removed D3, D4, D5: (no value), SparkFun-DiscreteSemi:DIODE-1N4148
- removed L1: 1R (40mH), rcl:0207/5V
- removed Q4, Q6: 2N3904, 808_lt:TO92
- removed R14: 2M2, rcl:0207/7
- removed R15: 50KB, TR808clone:B64Y
- removed R16: 47k, rcl:0207/7
- removed R17: 470k, rcl:0207/7
- removed TB: 22-23-2071, con-molex:22-23-2071
- added C3: 10n, rcl:C050-025X075
- added Q3: 2N3904, 808_lt:TO92
- added R11: 4k7, rcl:0207/10
- added R7: 15k, rcl:0207/10
- added SD: 22-23-2051, con-molex:22-23-2051
- C1: value 27n -> 10n
- C4: value 56n -> 5n6
- C5: value 10n -> 100p
- C6: value 33n -> 22n
- D1, D2: value (none) -> 1N4148DO35-7; device SparkFun-DiscreteSemi:DIODE-1N4148 -> diode:DO35-7
- R1: value 56k -> 270k; device rcl:0207/5V -> rcl:0207/10
- R10: value 820k -> 15k; device rcl:0207/7 -> rcl:0207/10
- R12: value 10k -> 1M5; device rcl:0207/7 -> rcl:0207/10
- R3: value 10k -> 220k; device rcl:0207/7 -> rcl:0207/10
- R5: value 270k -> 470k; device rcl:0207/7 -> rcl:0207/10
- R6: value 270k -> 820k; device rcl:0207/7 -> rcl:0207/10
- R8: value 270k -> 68k; device rcl:0207/7 -> rcl:0207/10
- R9: value 820k -> 1M; device rcl:0207/7 -> rcl:0207/10
- moved R12 174.8 mm to (6.35, -124.5), turned to 0 degrees
- moved C6 157.4 mm to (5.08, -116.8)
- moved C5 151.9 mm to (5.08, -88.9), turned to 0 degrees
- moved R10 151.5 mm to (6.35, -101.6), turned to 0 degrees
- moved R9 136.2 mm to (6.35, -96.5), turned to 0 degrees
- moved C4 134.4 mm to (5.08, -81.3)
- moved C1 112.9 mm to (5.08, -66.0), turned to 0 degrees
- moved Q1 105.5 mm to (3.81, -59.7), turned to 0 degrees
- moved R8 98.4 mm to (6.35, -54.6), turned to 0 degrees
- moved R3 86.6 mm to (6.35, -34.3), turned to 0 degrees
- moved R5 81.0 mm to (6.35, -39.4)
- moved R6 78.6 mm to (6.35, -44.5)
- moved R1 65.6 mm to (6.35, -15.2)
- moved D2 64.7 mm to (6.35, -26.7)
- moved D1 61.8 mm to (6.35, -20.3)
Connections:
- removed net N$10: Q6.2, R16.1, R17.2
- removed net N$14: Q4.2, R10.1, R8.2, R9.2
- removed net N$17: C5.2, R15.S
- removed net N$20: C1.1, Q1.1, R3.2
- removed net N$21: Q1.2, R1.2
- removed net N$22: C1.2, D1.C, D3.C, R5.1
- removed net N$23: D3.A, R8.1
- removed net N$24: R1.1, TB.1
- removed net N$25: D1.A, D2.A, TB.3
- new net N$12: C6.2, R12.1
- new net N$13: C7.1, R12.2
- new net N$8: C1.1, C3.1, R7.1
- net +12V: now also R11.1, R6.2, SD.3; no longer C6.1, L1.1, R10.2, R12.1, R15.A, R3.1, TB.5
- net GND: now also Q3.3, R1.2, R10.2, R8.2, SD.4; no longer C4.2, Q1.3, Q4.3, Q6.3, R17.1, R5.2, R6.2, TB.6
- net N$1: now also D1.A, R3.1; no longer C2.2, D2.C, D4.C, R6.1
- net N$11: now also SD.1; no longer TB.2
- net N$2: now also C2.2, D1.C, D2.C, R1.1; no longer D4.A, R9.1
- net N$3: now also D2.A, R5.1; no longer R15.E, TB.4
- net N$4: now also R3.2, R7.2, R8.1; no longer C4.1, D5.C, R14.1
- net N$5: now also C3.2, C5.2, C6.1, Q3.1, R11.2, R9.1; no longer C5.1, R14.2, R16.2
- net N$6: now also C1.2, C4.1, R10.1; no longer C6.2, C7.1, L1.2, Q6.1
- net N$7: now also SD.5; no longer TB.7
- net N$9: now also C4.2, C5.1, Q3.2, R9.2; no longer D5.A, Q4.1, R12.2
Routing:
- net GND: track 129.5 -> 41.5 mm
- net N$25: track 24.2 -> 0.00 mm
- net +12V: track 108.6 -> 86.9 mm
- net N$3: track 21.0 -> 0.00 mm
- net N$17: track 13.4 -> 0.00 mm
- net N$6: track 9.95 -> 0.00 mm
- net N$24: track 9.75 -> 0.00 mm
- net N$14: track 9.55 -> 0.00 mm
- net N$1: track 9.47 -> 0.00 mm
- net N$22: track 9.41 -> 0.00 mm
- net N$9: track 8.40 -> 0.00 mm
- net N$11: track 27.7 -> 19.5 mm
- net N$20: track 8.16 -> 0.00 mm
- net N$4: track 7.85 -> 0.00 mm
- net N$5: track 7.08 -> 0.00 mm
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