File: eagle/CR78-SD.brd (EAGLE design)
At the start: 100 x 80 mm, 46 parts, among them Q1 2N3904, Q2 2N3904, Q3 2N3904, Q4 2N3904, Q7 2N3904

Commit message: schemo
Routing:
- net +12V: track 86.9 -> 0.00 mm
- net N$7: track 42.8 -> 0.00 mm, vias 2 -> 0
- net GND: track 41.5 -> 0.00 mm
- net N$16: track 27.9 -> 0.00 mm
- net N$46: track 20.5 -> 0.00 mm
- net N$11: track 19.5 -> 0.00 mm
- net N$18: track 17.8 -> 0.00 mm
- net N$19: track 6.08 -> 0.00 mm
- net N$47: track 3.45 -> 0.00 mm
- net N$15: track 2.80 -> 0.00 mm

Commit message: layout begun
Parts:
- R1, R10, R11, R12, R13, R17, R3, R4, R5, R6, R8, R9: device rcl:0207/10 -> rcl:0204/7
- R2: device rcl:0207/5V -> rcl:0207/7
- moved R23 272.3 mm to (71.1, 57.1)
- moved C13 260.3 mm to (62.2, 54.6), turned to 270 degrees
- moved R17 240.0 mm to (71.1, 53.3)
- moved R22 239.0 mm to (64.8, 40.6), turned to 90 degrees
- moved C12 238.7 mm to (64.8, 48.3), turned to 180 degrees
- moved Q4 233.0 mm to (73.7, 49.5), turned to 180 degrees
- moved R16 222.9 mm to (73.7, 44.5), turned to 180 degrees
- moved C11 209.2 mm to (72.4, 38.1), turned to 180 degrees
- moved R15 208.5 mm to (73.7, 41.9), turned to 180 degrees
- moved R14 196.2 mm to (77.5, 33.0), turned to 90 degrees
- moved C10 195.8 mm to (81.3, 38.1), turned to 90 degrees
- moved R12 192.5 mm to (80.0, 53.3), turned to 90 degrees
- moved C6 179.5 mm to (83.8, 44.5), turned to 180 degrees
- moved D3 179.0 mm to (81.3, 27.9), turned to 270 degrees
- moved Q3 172.1 mm to (92.7, 40.6), turned to 180 degrees
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Connections:
- net N$23: now also C11.2

Commit message: 95pct auto
Parts:
- C9: device rcl:B45181A -> rcl:B45181B
- moved R2 21.1 mm to (28.4, 48.3)
- moved C2 19.9 mm to (34.3, 45.2)
- moved C9 17.7 mm to (30.2, 26.4), turned to 270 degrees
- moved Q2 17.3 mm to (27.9, 37.3)
- moved R21 17.3 mm to (30.0, 32.5)
- moved Q7 16.6 mm to (38.6, 27.4)
- moved Q1 15.9 mm to (62.2, 27.9)
- moved R17 15.9 mm to (57.1, 61.0)
- moved R19 15.9 mm to (39.4, 34.3)
- moved R23 15.9 mm to (57.1, 64.8)
- moved R8 15.9 mm to (62.2, 24.1)
- moved C12 15.9 mm to (50.8, 55.9), turned to 0 degrees
- moved R13 15.9 mm to (58.4, 33.0)
- moved R15 15.9 mm to (59.7, 49.5)
- moved C1 15.9 mm to (74.9, 27.9)
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
Commit message: last two routes
Parts:
- R1, R10, R11, R12, R13, R17, R3, R4, R5, R6, R8, R9: device rcl:0204/7 -> rcl:0207/7
- R14, R7: device rcl:0207/10 -> rcl:0207/7
- moved C3 15.3 mm to (77.5, 19.1), turned to 0 degrees
- moved R10 9.16 mm to (77.5, 35.6), turned to 0 degrees
- moved R17 8.98 mm to (50.8, 54.6)
- moved C4 7.41 mm to (77.5, 31.8), turned to 0 degrees
- moved R4 4.02 mm to (37.6, 52.1)
- moved C12 2.84 mm to (49.5, 58.4)
- moved R7 2.54 mm to (68.6, 20.3)
- moved C1 2.54 mm to (74.9, 25.4)
- moved C5 2.54 mm to (78.7, 25.4)
- moved C6 1.80 mm to (71.1, 53.3), turned to 90 degrees
- moved R1 1.80 mm to (50.8, 41.9)
- moved C13 1.27 mm to (49.5, 62.2), turned to 180 degrees
- moved C8 1.27 mm to (37.6, 39.1)
- moved R22 1.27 mm to (50.8, 49.5), turned to 0 degrees
- moved C9 1.27 mm to (31.5, 26.4)
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Routing:
- net GND: track 0.00 -> 211.1 mm
- net +12V: track 0.00 -> 119.5 mm
- net N$2: track 0.00 -> 53.9 mm
- net N$5: track 0.00 -> 44.7 mm
- net N$13: track 0.00 -> 40.5 mm
- net N$46: track 0.00 -> 38.8 mm
- net N$16: track 0.00 -> 27.9 mm
- net N$18: track 0.00 -> 24.1 mm
- net N$9: track 0.00 -> 22.6 mm
- net N$24: track 0.00 -> 21.8 mm
- net N$26: track 0.00 -> 16.8 mm
- net N$11: track 0.00 -> 11.9 mm
- net N$10: track 0.00 -> 10.7 mm
- net N$4: track 0.00 -> 10.4 mm
- net N$3: track 0.00 -> 9.94 mm
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
Commit message: routed and cutout
Parts:
- moved R18 34.6 mm to (10.7, 32.0), turned to 180 degrees
- moved C1 29.3 mm to (47.5, 15.2)
- moved C3 29.3 mm to (50.0, 8.89)
- moved C4 29.3 mm to (50.0, 21.6)
- moved D1 29.3 mm to (25.9, 8.89)
- moved R7 29.3 mm to (41.1, 10.2)
- moved R3 28.8 mm to (37.3, 7.62)
- moved C12 28.1 mm to (23.4, 48.3)
- moved R10 28.1 mm to (51.3, 25.4)
- moved C5 28.1 mm to (52.6, 15.2)
- moved R14 27.6 mm to (37.3, 31.8), turned to 180 degrees
- moved Q3 27.2 mm to (52.6, 40.6)
- moved R13 26.9 mm to (33.5, 22.9)
- moved C13 26.9 mm to (24.6, 52.1)
- moved R17 26.9 mm to (25.9, 44.5)
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Routing:
- net N$7: track 0.00 -> 52.2 mm
- net +12V: track 119.5 -> 153.4 mm
- net GND: track 211.1 -> 240.9 mm
- net N$46: track 38.8 -> 9.94 mm
- net N$19: track 0.00 -> 15.9 mm
- net N$13: track 40.5 -> 28.4 mm
- net N$2: track 53.9 -> 42.0 mm
- net N$5: track 44.7 -> 38.2 mm
- net N$3: track 9.94 -> 4.34 mm
- net N$16: track 27.9 -> 23.2 mm
- net N$11: track 11.9 -> 8.44 mm
- net N$15: track 6.58 -> 3.22 mm
- net N$18: track 24.1 -> 27.0 mm
- net N$17: track 8.67 -> 6.29 mm
- net N$20: track 8.15 -> 10.3 mm
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Other:
- board size 100 x 80 mm -> 100.8 x 80.8 mm

Commit message: tweaked smaller
Parts:
- moved Q7 1.85 mm to (15.7, 16.8), turned to 0 degrees
- moved C10 1.27 mm to (43.7, 34.3)
- moved C11 1.27 mm to (34.8, 34.3)
- moved C13 1.27 mm to (24.6, 50.8)
- moved C2 1.27 mm to (17.5, 36.8)
- moved C6 1.27 mm to (47.5, 41.9)
- moved Q3 1.27 mm to (52.6, 39.4)
- moved Q4 1.27 mm to (36.1, 45.7)
- moved R11 1.27 mm to (47.5, 31.8)
- moved R12 1.27 mm to (43.7, 48.3)
- moved R17 1.27 mm to (25.9, 43.2)
- moved R9 1.27 mm to (51.3, 31.8)
- moved SD 1.27 mm to (8.13, 48.3)
- moved R5 1.27 mm to (29.7, 15.2)
- moved R6 1.27 mm to (32.3, 15.2)
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Routing:
- net N$15: track 3.22 -> 5.06 mm
- net GND: track 240.9 -> 239.2 mm
- net N$7: track 52.2 -> 51.1 mm
- net N$19: track 15.9 -> 14.8 mm
- net N$5: track 38.2 -> 37.2 mm
- net +12V: track 153.4 -> 154.3 mm
- net N$16: track 23.2 -> 24.0 mm
- net N$8: track 6.13 -> 5.63 mm
Other:
- board size 100.8 x 80.8 mm -> 100.8 x 80.5 mm
