File: eagle/CR78-SD.sch (EAGLE design)
At the start: 39 parts, among them Q1 2N3904, Q2 2N3904, Q4 2N3904, Q6 2N3904, Q7 2N3904

Commit message: more schemo
Parts:
- removed D3, D4, D5: (no value), SparkFun-DiscreteSemi:DIODE1N4148
- removed L1: 1R (40mH), rcl:L-US0207/5V
- removed Q4, Q6: 2N3904, 808_lt:2N3904
- removed R14: 2M2, rcl:R-US_0207/7
- removed R15: 50KB, TR808clone:TRIM_EU-B64Y
- removed R16: 47k, rcl:R-US_0207/7
- removed R17: 470k, rcl:R-US_0207/7
- removed TB: 22-23-2071, con-molex:22-23-2071
- added C3: 10n, rcl:C-US050-025X075
- added Q3: 2N3904, 808_lt:2N3904
- added R11: 4k7, rcl:R-US_0207/10
- added R7: 15k, rcl:R-US_0207/10
- added SD: 22-23-2051, con-molex:22-23-2051
- C1: value 27n -> 10n
- C4: value 56n -> 5n6
- C5: value 10n -> 100p
- C6: value 33n -> 22n
- D1, D2: value (none) -> 1N4148DO35-7; device SparkFun-DiscreteSemi:DIODE1N4148 -> diode:1N4148DO35-7
- R1: value 56k -> 270k; device rcl:R-US_0207/5V -> rcl:R-US_0207/10
- R10: value 820k -> 15k; device rcl:R-US_0207/7 -> rcl:R-US_0207/10
- R12: value 10k -> 1M5; device rcl:R-US_0207/7 -> rcl:R-US_0207/10
- R3: value 10k -> 220k; device rcl:R-US_0207/7 -> rcl:R-US_0207/10
- R5: value 270k -> 470k; device rcl:R-US_0207/7 -> rcl:R-US_0207/10
- R6: value 270k -> 820k; device rcl:R-US_0207/7 -> rcl:R-US_0207/10
- R8: value 270k -> 68k; device rcl:R-US_0207/7 -> rcl:R-US_0207/10
- R9: value 820k -> 1M; device rcl:R-US_0207/7 -> rcl:R-US_0207/10
Connections:
- removed net N$10: Q6.B, R16.1, R17.2
- removed net N$14: Q4.B, R10.1, R8.2, R9.2
- removed net N$17: C5.2, R15.S
- removed net N$20: C1.1, Q1.C, R3.2
- removed net N$21: Q1.B, R1.2
- removed net N$22: C1.2, D1.C, D3.C, R5.1
- removed net N$23: D3.A, R8.1
- removed net N$24: R1.1, TB-1.S
- removed net N$25: D1.A, D2.A, TB-3.S
- new net N$12: C6.2, R12.1
- new net N$13: C7.1, R12.2
- new net N$8: C1.1, C3.1, R7.1
- net +12V: now also R11.1, R6.2, SD-3.S; no longer C6.1, L1.1, R10.2, R12.1, R15.A, R3.1, TB-5.S
- net GND: now also Q3.E, R1.2, R10.2, R8.2, SD-4.S; no longer C4.2, Q1.E, Q4.E, Q6.E, R17.1, R5.2, R6.2, TB-6.S
- net N$1: now also D1.A, R3.1; no longer C2.2, D2.C, D4.C, R6.1
- net N$11: now also SD-1.S; no longer TB-2.S
- net N$2: now also C2.2, D1.C, D2.C, R1.1; no longer D4.A, R9.1
- net N$3: now also D2.A, R5.1; no longer R15.E, TB-4.S
- net N$4: now also R3.2, R7.2, R8.1; no longer C4.1, D5.C, R14.1
- net N$5: now also C3.2, C5.2, C6.1, Q3.C, R11.2, R9.1; no longer C5.1, R14.2, R16.2
- net N$6: now also C1.2, C4.1, R10.1; no longer C6.2, C7.1, L1.2, Q6.C
- net N$7: now also SD-5.S; no longer TB-7.S
- net N$9: now also C4.2, C5.1, Q3.B, R9.2; no longer D5.A, Q4.C, R12.2
Other:
- note removed: "NOISE"
- moved on the sheet: C1, C4, C5, C6, Q1, R1, R10, R12, R3, R5, R6, R8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
