File: eagle/CR78-SD.sch (EAGLE design)
At the start: 46 parts, among them Q1 2N3904, Q2 2N3904, Q3 2N3904, Q4 2N3904, Q7 2N3904

Commit message: schemo
Other:
- moved on the sheet: SD-3, SD-4
Changed lines of the file:
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@@
 <instance part="SD" gate="-1" x="0" y="68.58" rot="R180"/>
 <instance part="SD" gate="-2" x="83.82" y="7.62" rot="R180"/>
-<instance part="SD" gate="-3" x="20.32" y="114.3"/>
-<instance part="SD" gate="-4" x="20.32" y="111.76"/>
+<instance part="SD" gate="-3" x="7.62" y="93.98"/>
+<instance part="SD" gate="-4" x="7.62" y="91.44"/>
 <instance part="SD" gate="-5" x="198.12" y="81.28" rot="R180"/>
-<instance part="P+11" gate="1" x="12.7" y="124.46"/>
-<instance part="GND18" gate="1" x="12.7" y="104.14"/>
+<instance part="P+11" gate="1" x="0" y="104.14"/>
+<instance part="GND18" gate="1" x="0" y="83.82"/>
 <instance part="R1" gate="G$1" x="43.18" y="66.04" rot="R270"/>
 <instance part="D1" gate="G$1" x="55.88" y="73.66" rot="R180"/>
@@
 <segment>
 <pinref part="P+11" gate="1" pin="+12V"/>
-<wire x1="12.7" y1="114.3" x2="12.7" y2="121.92" width="0.1524" layer="91"/>
+<wire x1="0" y1="93.98" x2="0" y2="101.6" width="0.1524" layer="91"/>
 <pinref part="SD" gate="-3" pin="S"/>
-<wire x1="17.78" y1="114.3" x2="12.7" y2="114.3" width="0.1524" layer="91"/>
+<wire x1="5.08" y1="93.98" x2="0" y2="93.98" width="0.1524" layer="91"/>
 </segment>
 <segment>
@@
 <pinref part="SD" gate="-4" pin="S"/>
 <pinref part="GND18" gate="1" pin="GND"/>
-<wire x1="17.78" y1="111.76" x2="12.7" y2="111.76" width="0.1524" layer="91"/>
-<wire x1="12.7" y1="111.76" x2="12.7" y2="106.68" width="0.1524" layer="91"/>
+<wire x1="5.08" y1="91.44" x2="0" y2="91.44" width="0.1524" layer="91"/>
+<wire x1="0" y1="91.44" x2="0" y2="86.36" width="0.1524" layer="91"/>
 </segment>
 <segment>

Commit message: layout begun
Parts:
- R1, R10, R11, R12, R13, R17, R3, R4, R5, R6, R8, R9: device rcl:R-US_0207/10 -> rcl:R-US_0204/7
- R2: device rcl:R-US_0207/5V -> rcl:R-US_0207/7
Connections:
- net N$23: now also C11.2
Changed lines of the file:
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@@
 <grid distance="0.1" unitdist="inch" unit="inch" style="lines" multiple="1" display="no" altdistance="0.01" altunitdist="inch" altunit="inch"/>
 <layers>
-<layer number="1" name="Top" color="4" fill="1" visible="no" active="no"/>
-<layer number="16" name="Bottom" color="1" fill="1" visible="no" active="no"/>
-<layer number="17" name="Pads" color="2" fill="1" visible="no" active="no"/>
-<layer number="18" name="Vias" color="2" fill="1" visible="no" active="no"/>
-<layer number="19" name="Unrouted" color="6" fill="1" visible="no" active="no"/>
-<layer number="20" name="Dimension" color="15" fill="1" visible="no" active="no"/>
-<layer number="21" name="tPlace" color="7" fill="1" visible="no" active="no"/>
-<layer number="22" name="bPlace" color="7" fill="1" visible="no" active="no"/>
-<layer number="23" name="tOrigins" color="15" fill="1" visible="no" active="no"/>
-<layer number="24" name="bOrigins" color="15" fill="1" visible="no" active="no"/>
-<layer number="25" name="tNames" color="7" fill="1" visible="no" active="no"/>
-<layer number="26" name="bNames" color="7" fill="1" visible="no" active="no"/>
-<layer number="27" name="tValues" color="7" fill="1" visible="no" active="no"/>
-<layer number="28" name="bValues" color="7" fill="1" visible="no" active="no"/>
+<layer number="1" name="Top" color="4" fill="1" visible="yes" active="no"/>
+<layer number="16" name="Bottom" color="1" fill="1" visible="yes" active="no"/>
+<layer number="17" name="Pads" color="2" fill="1" visible="yes" active="no"/>
+<layer number="18" name="Vias" color="2" fill="1" visible="yes" active="no"/>
+<layer number="19" name="Unrouted" color="6" fill="1" visible="yes" active="no"/>
+<layer number="20" name="Dimension" color="15" fill="1" visible="yes" active="no"/>
+<layer number="21" name="tPlace" color="7" fill="1" visible="yes" active="no"/>
+<layer number="22" name="bPlace" color="7" fill="1" visible="yes" active="no"/>
+<layer number="23" name="tOrigins" color="15" fill="1" visible="yes" active="no"/>
+<layer number="24" name="bOrigins" color="15" fill="1" visible="yes" active="no"/>
+<layer number="25" name="tNames" color="7" fill="1" visible="yes" active="no"/>
+<layer number="26" name="bNames" color="7" fill="1" visible="yes" active="no"/>
+<layer number="27" name="tValues" color="7" fill="1" visible="yes" active="no"/>
+<layer number="28" name="bValues" color="7" fill="1" visible="yes" active="no"/>
 <layer number="29" name="tStop" color="7" fill="3" visible="no" active="no"/>
 <layer number="30" name="bStop" color="7" fill="6" visible="no" active="no"/>
@@
 <layer number="35" name="tGlue" color="7" fill="4" visible="no" active="no"/>
 <layer number="36" name="bGlue" color="7" fill="5" visible="no" active="no"/>
-<layer number="37" name="tTest" color="7" fill="1" visible="no" active="no"/>
-<layer number="38" name="bTest" color="7" fill="1" visible="no" active="no"/>
+<layer number="37" name="tTest" color="7" fill="1" visible="yes" active="no"/>
+<layer number="38" name="bTest" color="7" fill="1" visible="yes" active="no"/>
 <layer number="39" name="tKeepout" color="4" fill="11" visible="no" active="no"/>
 <layer number="40" name="bKeepout" color="1" fill="11" visible="no" active="no"/>
@@
 <layer number="44" name="Drills" color="7" fill="1" visible="no" active="no"/>
 <layer number="45" name="Holes" color="7" fill="1" visible="no" active="no"/>
-<layer number="46" name="Milling" color="3" fill="1" visible="no" active="no"/>
-<layer number="47" name="Measures" color="7" fill="1" visible="no" active="no"/>
-<layer number="48" name="Document" color="7" fill="1" visible="no" active="no"/>
-<layer number="49" name="Reference" color="7" fill="1" visible="no" active="no"/>
-<layer number="50" name="dxf" color="7" fill="1" visible="no" active="no"/>
-<layer number="51" name="tDocu" color="7" fill="1" visible="no" active="no"/>
-<layer number="52" name="bDocu" color="7" fill="1" visible="no" active="no"/>
-<layer number="53" name="tGND_GNDA" color="7" fill="9" visible="no" active="no"/>
-<layer number="54" name="bGND_GNDA" color="1" fill="9" visible="no" active="no"/>
-<layer number="56" name="wert" color="7" fill="1" visible="no" active="no"/>
-<layer number="57" name="tCAD" color="7" fill="1" visible="no" active="no"/>
-<layer number="59" name="tCarbon" color="7" fill="1" visible="no" active="no"/>
-<layer number="60" name="bCarbon" color="7" fill="1" visible="no" active="no"/>
+<layer number="46" name="Milling" color="3" fill="1" visible="yes" active="no"/>
+<layer number="47" name="Measures" color="7" fill="1" visible="yes" active="no"/>
+<layer number="48" name="Document" color="7" fill="1" visible="yes" active="no"/>
+<layer number="49" name="Reference" color="7" fill="1" visible="yes" active="no"/>
+<layer number="50" name="dxf" color="7" fill="1" visible="yes" active="no"/>
+<layer number="51" name="tDocu" color="7" fill="1" visible="yes" active="no"/>
+<layer number="52" name="bDocu" color="7" fill="1" visible="yes" active="no"/>
+<layer number="53" name="tGND_GNDA" color="7" fill="9" visible="yes" active="no"/>
+<layer number="54" name="bGND_GNDA" color="1" fill="9" visible="yes" active="no"/>
+<layer number="56" name="wert" color="7" fill="1" visible="yes" active="no"/>
+<layer number="57" name="tCAD" color="7" fill="1" visible="yes" active="no"/>
+<layer number="59" name="tCarbon" color="7" fill="1" visible="yes" active="no"/>
+<layer number="60" name="bCarbon" color="7" fill="1" visible="yes" active="no"/>
 <layer number="90" name="Modules" color="5" fill="1" visible="yes" active="yes"/>
 <layer number="91" name="Nets" color="2" fill="1" visible="yes" active="yes"/>
@@
 <part name="GND3" library="supply1" deviceset="GND" device=""/>
 <part name="P+3" library="supply1" deviceset="+12V" device=""/>
-<part name="R4" library="rcl" deviceset="R-US_" device="0207/10" value="10k"/>
-<part name="R2" library="rcl" deviceset="R-US_" device="0207/5V" value="56k"/>
+<part name="R4" library="rcl" deviceset="R-US_" device="0204/7" value="10k"/>
+<part name="R2" library="rcl" deviceset="R-US_" device="0207/7" value="56k"/>
 <part name="C2" library="rcl" deviceset="C-US" device="050-025X075" value="27n"/>
 <part name="P+6" library="supply1" deviceset="+12V" device=""/>
@@
 <part name="P+11" library="supply1" deviceset="+12V" device=""/>
 <part name="GND18" library="supply1" deviceset="GND" device=""/>
-<part name="R1" library="rcl" deviceset="R-US_" device="0207/10" value="270k"/>
+<part name="R1" library="rcl" deviceset="R-US_" device="0204/7" value="270k"/>
 <part name="D1" library="diode" deviceset="1N4148" device="DO35-7"/>
 <part name="D2" library="diode" deviceset="1N4148" device="DO35-7"/>
-<part name="R3" library="rcl" deviceset="R-US_" device="0207/10" value="220k"/>
-<part name="R5" library="rcl" deviceset="R-US_" device="0207/10" value="470k"/>
-<part name="R6" library="rcl" deviceset="R-US_" device="0207/10" value="820k"/>
+<part name="R3" library="rcl" deviceset="R-US_" device="0204/7" value="220k"/>
+<part name="R5" library="rcl" deviceset="R-US_" device="0204/7" value="470k"/>
+<part name="R6" library="rcl" deviceset="R-US_" device="0204/7" value="820k"/>
 <part name="GND1" library="supply1" deviceset="GND" device=""/>
 <part name="R7" library="rcl" deviceset="R-US_" device="0207/10" value="15k"/>
-<part name="R8" library="rcl" deviceset="R-US_" device="0207/10" value="68k"/>
+<part name="R8" library="rcl" deviceset="R-US_" device="0204/7" value="68k"/>
 <part name="Q1" library="808_lt" deviceset="2N3904" device=""/>
 <part name="GND2" library="supply1" deviceset="GND" device=""/>
@@
 <part name="C4" library="rcl" deviceset="C-US" device="050-025X075" value="5n6"/>
 <part name="C5" library="rcl" deviceset="C-US" device="050-025X075" value="100p"/>
-<part name="R9" library="rcl" deviceset="R-US_" device="0207/10" value="1M"/>
-<part name="R10" library="rcl" deviceset="R-US_" device="0207/10" value="15k"/>
+<part name="R9" library="rcl" deviceset="R-US_" device="0204/7" value="1M"/>
+<part name="R10" library="rcl" deviceset="R-US_" device="0204/7" value="15k"/>
 <part name="GND4" library="supply1" deviceset="GND" device=""/>
 <part name="Q3" library="808_lt" deviceset="2N3904" device=""/>
-<part name="R11" library="rcl" deviceset="R-US_" device="0207/10" value="4k7"/>
+<part name="R11" library="rcl" deviceset="R-US_" device="0204/7" value="4k7"/>
 <part name="P+1" library="supply1" deviceset="+12V" device=""/>
 <part name="GND5" library="supply1" deviceset="GND" device=""/>
 <part name="C6" library="rcl" deviceset="C-US" device="050-025X075" value="22n"/>
-<part name="R12" library="rcl" deviceset="R-US_" device="0207/10" value="1M5"/>
-<part name="R13" library="rcl" deviceset="R-US_" device="0207/10" value="10k"/>
+<part name="R12" library="rcl" deviceset="R-US_" device="0204/7" value="1M5"/>
+<part name="R13" library="rcl" deviceset="R-US_" device="0204/7" value="10k"/>
 <part name="P+4" library="supply1" deviceset="+12V" device=""/>
 <part name="GND6" library="supply1" deviceset="GND" device=""/>
@@
 <part name="R16" library="rcl" deviceset="R-US_" device="0207/7" value="470k"/>
 <part name="Q4" library="808_lt" deviceset="2N3904" device=""/>
-<part name="R17" library="rcl" deviceset="R-US_" device="0207/10" value="2k7"/>
+<part name="R17" library="rcl" deviceset="R-US_" device="0204/7" value="2k7"/>
 <part name="C12" library="rcl" deviceset="C-US" device="050-025X075" value="5n6"/>
 <part name="GND8" library="supply1" deviceset="GND" device=""/>
@@
 <pinref part="R22" gate="1" pin="S"/>
 <wire x1="104.14" y1="12.7" x2="104.14" y2="17.78" width="0.1524" layer="91"/>
-</segment>
-</net>
+<pinref part="C11" gate="G$1" pin="2"/>
+</segment>
+</net>

Commit message: 95pct auto
Parts:
- C9: device rcl:CPOL-USB45181A -> rcl:CPOL-USB45181B
Changed lines of the file:
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@@
 <part name="R20" library="rcl" deviceset="R-US_" device="0207/7" value="47k"/>
 <part name="R21" library="rcl" deviceset="R-US_" device="0207/7" value="220R"/>
-<part name="C9" library="rcl" deviceset="CPOL-US" device="B45181A" value="1uF"/>
+<part name="C9" library="rcl" deviceset="CPOL-US" device="B45181B" value="1uF"/>
 <part name="JCK1" library="erthenvar" deviceset="AUDIO-JACK" device=""/>
 <part name="GND15" library="supply1" deviceset="GND" device=""/>

Commit message: last two routes
Parts:
- R1, R10, R11, R12, R13, R17, R3, R4, R5, R6, R8, R9: device rcl:R-US_0204/7 -> rcl:R-US_0207/7
- R14, R7: device rcl:R-US_0207/10 -> rcl:R-US_0207/7
Changed lines of the file:
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@@
 <part name="GND3" library="supply1" deviceset="GND" device=""/>
 <part name="P+3" library="supply1" deviceset="+12V" device=""/>
-<part name="R4" library="rcl" deviceset="R-US_" device="0204/7" value="10k"/>
+<part name="R4" library="rcl" deviceset="R-US_" device="0207/7" value="10k"/>
 <part name="R2" library="rcl" deviceset="R-US_" device="0207/7" value="56k"/>
 <part name="C2" library="rcl" deviceset="C-US" device="050-025X075" value="27n"/>
@@
 <part name="P+11" library="supply1" deviceset="+12V" device=""/>
 <part name="GND18" library="supply1" deviceset="GND" device=""/>
-<part name="R1" library="rcl" deviceset="R-US_" device="0204/7" value="270k"/>
+<part name="R1" library="rcl" deviceset="R-US_" device="0207/7" value="270k"/>
 <part name="D1" library="diode" deviceset="1N4148" device="DO35-7"/>
 <part name="D2" library="diode" deviceset="1N4148" device="DO35-7"/>
-<part name="R3" library="rcl" deviceset="R-US_" device="0204/7" value="220k"/>
-<part name="R5" library="rcl" deviceset="R-US_" device="0204/7" value="470k"/>
-<part name="R6" library="rcl" deviceset="R-US_" device="0204/7" value="820k"/>
+<part name="R3" library="rcl" deviceset="R-US_" device="0207/7" value="220k"/>
+<part name="R5" library="rcl" deviceset="R-US_" device="0207/7" value="470k"/>
+<part name="R6" library="rcl" deviceset="R-US_" device="0207/7" value="820k"/>
 <part name="GND1" library="supply1" deviceset="GND" device=""/>
-<part name="R7" library="rcl" deviceset="R-US_" device="0207/10" value="15k"/>
-<part name="R8" library="rcl" deviceset="R-US_" device="0204/7" value="68k"/>
+<part name="R7" library="rcl" deviceset="R-US_" device="0207/7" value="15k"/>
+<part name="R8" library="rcl" deviceset="R-US_" device="0207/7" value="68k"/>
 <part name="Q1" library="808_lt" deviceset="2N3904" device=""/>
 <part name="GND2" library="supply1" deviceset="GND" device=""/>
@@
 <part name="C4" library="rcl" deviceset="C-US" device="050-025X075" value="5n6"/>
 <part name="C5" library="rcl" deviceset="C-US" device="050-025X075" value="100p"/>
-<part name="R9" library="rcl" deviceset="R-US_" device="0204/7" value="1M"/>
-<part name="R10" library="rcl" deviceset="R-US_" device="0204/7" value="15k"/>
+<part name="R9" library="rcl" deviceset="R-US_" device="0207/7" value="1M"/>
+<part name="R10" library="rcl" deviceset="R-US_" device="0207/7" value="15k"/>
 <part name="GND4" library="supply1" deviceset="GND" device=""/>
 <part name="Q3" library="808_lt" deviceset="2N3904" device=""/>
-<part name="R11" library="rcl" deviceset="R-US_" device="0204/7" value="4k7"/>
+<part name="R11" library="rcl" deviceset="R-US_" device="0207/7" value="4k7"/>
 <part name="P+1" library="supply1" deviceset="+12V" device=""/>
 <part name="GND5" library="supply1" deviceset="GND" device=""/>
 <part name="C6" library="rcl" deviceset="C-US" device="050-025X075" value="22n"/>
-<part name="R12" library="rcl" deviceset="R-US_" device="0204/7" value="1M5"/>
-<part name="R13" library="rcl" deviceset="R-US_" device="0204/7" value="10k"/>
+<part name="R12" library="rcl" deviceset="R-US_" device="0207/7" value="1M5"/>
+<part name="R13" library="rcl" deviceset="R-US_" device="0207/7" value="10k"/>
 <part name="P+4" library="supply1" deviceset="+12V" device=""/>
 <part name="GND6" library="supply1" deviceset="GND" device=""/>
@@
 <part name="C10" library="rcl" deviceset="C-US" device="050-025X075" value="18n"/>
 <part name="GND7" library="supply1" deviceset="GND" device=""/>
-<part name="R14" library="rcl" deviceset="R-US_" device="0207/10" value="1M5"/>
+<part name="R14" library="rcl" deviceset="R-US_" device="0207/7" value="1M5"/>
 <part name="R15" library="rcl" deviceset="R-US_" device="0207/7" value="47k"/>
 <part name="C11" library="rcl" deviceset="C-US" device="050-025X075" value="8n2"/>
 <part name="R16" library="rcl" deviceset="R-US_" device="0207/7" value="470k"/>
 <part name="Q4" library="808_lt" deviceset="2N3904" device=""/>
-<part name="R17" library="rcl" deviceset="R-US_" device="0204/7" value="2k7"/>
+<part name="R17" library="rcl" deviceset="R-US_" device="0207/7" value="2k7"/>
 <part name="C12" library="rcl" deviceset="C-US" device="050-025X075" value="5n6"/>
 <part name="GND8" library="supply1" deviceset="GND" device=""/>
